Commit message: Create CVC Ros node

File: convex_clustering_description/urdf/base_velodyne.urdf.xacro (robot description, xacro)
@@ -168,10 +168,10 @@
     </VLP-16> -->
     <xacro:include filename="$(find velodyne_description)/urdf/VLP-16.urdf.xacro"/>
-    <VLP-16 parent="base_link" name="velodyne_front" topic="/velodyne_points_front" hz="10" samples="440" gpu="${gpu}">
-        <origin xyz="0.3 0 0.55" rpy="0 0 0" />
+    <VLP-16 parent="base_link" name="velodyne_front" topic="/velodyne_points" hz="10" samples="440" gpu="${gpu}">
+        <origin xyz="0 0 0.55" rpy="0 0 0" />
     </VLP-16>
-    <VLP-16 parent="base_link" name="velodyne_rear" topic="/velodyne_points_rear" hz="10" samples="440" gpu="${gpu}">
+    <!-- <VLP-16 parent="base_link" name="velodyne_rear" topic="/velodyne_points_rear" hz="10" samples="440" gpu="${gpu}">
         <origin xyz="-0.3 0 0.55" rpy="0 0 3.1415" />
-    </VLP-16>
+    </VLP-16> -->
     <!-- Front sonar sensor -->
     <link name="base_sonar_front">

Commit message: Add Rviz Visualization

File: convex_clustering_description/urdf/base_velodyne.urdf.xacro (robot description, xacro)
@@ -171,7 +171,7 @@
         <origin xyz="0 0 0.55" rpy="0 0 0" />
     </VLP-16>
-    <!-- <VLP-16 parent="base_link" name="velodyne_rear" topic="/velodyne_points_rear" hz="10" samples="440" gpu="${gpu}">
-        <origin xyz="-0.3 0 0.55" rpy="0 0 3.1415" />
-    </VLP-16> -->
+    <VLP-16 parent="base_link" name="velodyne_rear" topic="/velodyne_points_rear" hz="10" samples="440" gpu="${gpu}">
+        <origin xyz="2 2 0.55" rpy="0 0 3.1415" />
+    </VLP-16>
     <!-- Front sonar sensor -->
     <link name="base_sonar_front">

Commit message: Change Centroid Method

File: convex_clustering_description/urdf/base_velodyne.urdf.xacro (robot description, xacro)
@@ -165,11 +165,11 @@
     <!-- <xacro:include filename="$(find velodyne_description)/urdf/VLP-16.urdf.xacro"/>
     <VLP-16 parent="base_link" name="velodyne_front" topic="/velodyne_points_front" hz="10" samples="440" gpu="${gpu}">
-        <origin xyz="0 0 0.55" rpy="0 0 0" />
+        <origin xyz="0 0 0.55" rpy="s0 0 0" />
     </VLP-16> -->
     <xacro:include filename="$(find velodyne_description)/urdf/VLP-16.urdf.xacro"/>
-    <VLP-16 parent="base_link" name="velodyne_front" topic="/velodyne_points" hz="10" samples="440" gpu="${gpu}">
+    <VLP-16 parent="base_link" name="velodyne_front" topic="/velodyne_points_1" hz="10" samples="440" gpu="${gpu}">
         <origin xyz="0 0 0.55" rpy="0 0 0" />
     </VLP-16>
-    <VLP-16 parent="base_link" name="velodyne_rear" topic="/velodyne_points_rear" hz="10" samples="440" gpu="${gpu}">
+    <VLP-16 parent="base_link" name="velodyne_rear" topic="/velodyne_points_2" hz="10" samples="440" gpu="${gpu}">
         <origin xyz="2 2 0.55" rpy="0 0 3.1415" />
     </VLP-16>

Commit message: Add Centroid Merge

File: convex_clustering_description/urdf/base_velodyne.urdf.xacro (robot description, xacro)
@@ -172,5 +172,5 @@
     </VLP-16>
     <VLP-16 parent="base_link" name="velodyne_rear" topic="/velodyne_points_2" hz="10" samples="440" gpu="${gpu}">
-        <origin xyz="2 2 0.55" rpy="0 0 3.1415" />
+        <origin xyz="2 2 0.55" rpy="0 0 3.1415" /> <!-- 3.1415 -->
     </VLP-16>
     <!-- Front sonar sensor -->
