Commit message: Add description

File: curved_clustering_description/urdf/base_velodyne.urdf.xacro (robot description, xacro)
@@ -5,6 +5,6 @@
        xmlns:xacro="http://ros.org/wiki/xacro"
        name="vehicle_v2" >
-    <xacro:include filename="$(find vrep_holonomic_description)/urdf/base_velodyne.gazebo.xacro"/>
-    <xacro:include filename="$(find vrep_holonomic_description)/urdf/materials.urdf.xacro"/>
+    <xacro:include filename="$(find curved_clustering_description)/urdf/base_velodyne.gazebo.xacro"/>
+    <xacro:include filename="$(find curved_clustering_description)/urdf/materials.urdf.xacro"/>
     <xacro:arg name="gpu" default="false"/>
     <xacro:property name="gpu" value="$(arg gpu)" />
@@ -21,5 +21,5 @@
             <origin xyz="0 0 0" rpy="0 0 0" />
             <geometry>
-                <mesh filename="package://vrep_holonomic_description/meshes/base_link.STL" />
+                <mesh filename="package://curved_clustering_description/meshes/base_link.STL" />
             </geometry>
             <material name="material_light_grey"/>
@@ -47,5 +47,5 @@
             <origin xyz="0 0 0" rpy="0 0 0" />
             <geometry>
-                <mesh filename="package://vrep_holonomic_description/meshes/br_wheel_link.STL" />
+                <mesh filename="package://curved_clustering_description/meshes/br_wheel_link.STL" />
             </geometry>
             <material name="material_orange"/>
@@ -74,5 +74,5 @@
             <origin xyz="0 0 0" rpy="0 0 0" />
             <geometry>
-                <mesh filename="package://vrep_holonomic_description/meshes/bl_wheel_link.STL" />
+                <mesh filename="package://curved_clustering_description/meshes/bl_wheel_link.STL" />
             </geometry>
             <material name="material_orange"/>
@@ -101,5 +101,5 @@
             <origin xyz="0 0 0" rpy="0 0 0" />
             <geometry>
-                <mesh filename="package://vrep_holonomic_description/meshes/fr_wheel_link.STL" />
+                <mesh filename="package://curved_clustering_description/meshes/fr_wheel_link.STL" />
             </geometry>
             <material name="material_orange"/>
@@ -128,5 +128,5 @@
             <origin xyz="0 0 0" rpy="0 0 0" />
             <geometry>
-                <mesh filename="package://vrep_holonomic_description/meshes/fl_wheel_link.STL" />
+                <mesh filename="package://curved_clustering_description/meshes/fl_wheel_link.STL" />
             </geometry>
             <material name="material_orange"/>
@@ -184,5 +184,5 @@
             <origin xyz="0 0 0" rpy="0 0 0" />
             <geometry>
-                <mesh filename="package://vrep_holonomic_description/meshes/max_sonar_ez4.dae"/>
+                <mesh filename="package://curved_clustering_description/meshes/max_sonar_ez4.dae"/>
             </geometry>
         </visual>
@@ -209,5 +209,5 @@
             <origin xyz="0 0 0" rpy="0 0 0" />
             <geometry>
-                <mesh filename="package://vrep_holonomic_description/meshes/max_sonar_ez4.dae"/>
+                <mesh filename="package://curved_clustering_description/meshes/max_sonar_ez4.dae"/>
             </geometry>
         </visual>
@@ -234,5 +234,5 @@
             <origin xyz="0 0 0" rpy="0 0 0" />
             <geometry>
-                <mesh filename="package://vrep_holonomic_description/meshes/max_sonar_ez4.dae"/>
+                <mesh filename="package://curved_clustering_description/meshes/max_sonar_ez4.dae"/>
             </geometry>
         </visual>
@@ -259,5 +259,5 @@
             <origin xyz="0 0 0" rpy="0 0 0" />
             <geometry>
-                <mesh filename="package://vrep_holonomic_description/meshes/max_sonar_ez4.dae"/>
+                <mesh filename="package://curved_clustering_description/meshes/max_sonar_ez4.dae"/>
             </geometry>
         </visual>
@@ -284,5 +284,5 @@
             <origin xyz="0.0 0.0 0.0" rpy="0 0 0" />
             <geometry>
-                <mesh filename="package://vrep_holonomic_description/meshes/kinect.dae"/>
+                <mesh filename="package://curved_clustering_description/meshes/kinect.dae"/>
             </geometry>
         </visual>
@@ -290,5 +290,5 @@
             <origin xyz="0.0 0.0 0.0" rpy="0 0 0" />
             <geometry>
-                <mesh filename="package://vrep_holonomic_description/meshes/kinect.dae"/>
+                <mesh filename="package://curved_clustering_description/meshes/kinect.dae"/>
             </geometry>
         </collision>
